File: Hardware/TP_MCU/TP_MCU.kicad_pcb (KiCad board)
At the start: 2 copper layers, 58 x 48 mm, 27 parts, among them J1 Conn_02x07_Odd_Even, J2 POWER, J3 INPUT, J4 OUTPUT, U1 BU33SD5WG-TR, U2 STM32L021K4Tx, U3 MCP4801-E/SN

Commit message: Add files via upload
Routing:
- net GND: vias 15 -> 20
Other:
- board text added: "Kévin OKONSKI et Jérôme DUPOUTS"
Changed lines of the file:
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@@
   (gr_arc (start 60 83.999999) (mid 57.189448 82.825173) (end 56.048812 80.000573) (layer "Edge.Cuts") (width 0.15))
   (gr_line (start 110 36) (end 110 36) (layer "Edge.Cuts") (width 0.15))
+  (gr_text "Kévin OKONSKI et Jérôme DUPOUTS" (at 85 81.7) (layer "F.Cu")
+    (effects (font (size 1.5 1.5) (thickness 0.3)))
+  )
   (dimension (type aligned) (layer "Cmts.User")
     (pts (xy 60 40) (xy 60 80))
@@
   (via (at 65.3 49.7) (size 1.2) (drill 0.6) (layers "F.Cu" "B.Cu") (free) (net 2))
   (via (at 73.1 54.1) (size 1.2) (drill 0.6) (layers "F.Cu" "B.Cu") (free) (net 2))
+  (via (at 72.7 76.6) (size 1.2) (drill 0.6) (layers "F.Cu" "B.Cu") (free) (net 2))
   (via (at 93.2 50.1) (size 1.2) (drill 0.6) (layers "F.Cu" "B.Cu") (free) (net 2))
+  (via (at 101.5 76) (size 1.2) (drill 0.6) (layers "F.Cu" "B.Cu") (free) (net 2))
   (via (at 79.7 53) (size 1.2) (drill 0.6) (layers "F.Cu" "B.Cu") (free) (net 2))
+  (via (at 93.4 40.9) (size 1.2) (drill 0.6) (layers "F.Cu" "B.Cu") (free) (net 2))
   (via (at 108.4 48.2) (size 1.2) (drill 0.6) (layers "F.Cu" "B.Cu") (free) (net 2))
   (via (at 89.2 54.2) (size 1.2) (drill 0.6) (layers "F.Cu" "B.Cu") (free) (net 2))
+  (via (at 86.9 49.8) (size 1.2) (drill 0.6) (layers "F.Cu" "B.Cu") (free) (net 2))
+  (via (at 98.3 58.5) (size 1.2) (drill 0.6) (layers "F.Cu" "B.Cu") (free) (net 2))
   (via (at 73.1 56.4) (size 1.2) (drill 0.6) (layers "F.Cu" "B.Cu") (free) (net 2))
   (via (at 67.5 72.2) (size 1.2) (drill 0.6) (layers "F.Cu" "B.Cu") (free) (net 2))
